Commit message: URDF is now taking into considration the dampers width

File: src/python/orm_r3.urdf (robot description, URDF)
Before this commit: robot orm_r3, 8 links, 7 joints
Joints:
- joint joint1: origin xyz=0 0.064 0.038 rpy=0 0 0 -> xyz=0 0.0655 0.038 rpy=0 0 0
- joint joint4: origin xyz=0 -0.041 -0.032 rpy=0 0 0 -> xyz=0 -0.0425 -0.0335 rpy=0 0 0
